File: pcb/nikon_gps/nikon_gps.sch (KiCad schematic (older format))
At the start: 34 parts, among them J1 Conn_01x03, SW1 ON/OFF, U1 Hornet ORG1411, U2 SN74LV1T126_ALT, U3 MAX16054, U4 MIC5205-3.3

Commit message: Readme and schematics update.
Parts:
- C6: value 470pF -> 1nF
- C8: value 4.7uF -> 10uF
- R9: value 330 -> 270
Changed lines of the file:
@@
 P 6600 5000
 F 0 "C8" H 6700 5000 50  0000 L CNN
-F 1 "4.7uF" H 6750 4900 50  0000 C CNN
+F 1 "10uF" H 6750 4900 50  0000 C CNN
 F 2 "Capacitors_SMD:C_0805" H 6600 5000 50  0001 C CNN
 F 3 "" H 6600 5000 50  0001 C CNN
@@
 P 8000 5000
 F 0 "C6" H 7850 5000 50  0000 C CNN
-F 1 "470pF" H 7850 4900 50  0000 C CNN
+F 1 "1nF" H 7850 4900 50  0000 C CNN
 F 2 "Capacitors_SMD:C_0603" H 8000 5000 50  0001 C CNN
 F 3 "" H 8000 5000 50  0001 C CNN
@@
 P 3000 4450
 F 0 "R9" H 3200 4400 50  0000 C CNN
-F 1 "330" H 3200 4500 50  0000 C CNN
+F 1 "270" H 3200 4500 50  0000 C CNN
 F 2 "Resistors_SMD:R_0805" V 2930 4450 50  0001 C CNN
 F 3 "" H 3000 4450 50  0001 C CNN
